Commit message: 5-15

File: legged_examples/legged_unitree/legged_unitree_description/urdf/robot.xacro (robot description, xacro)
@@ -7,17 +7,4 @@
     <xacro:include filename="$(find legged_unitree_description)/urdf/common/imu.xacro"/>
     <xacro:include filename="$(find legged_unitree_description)/urdf/$(arg robot_type)/const.xacro"/>
-    <!-- <link name="world">
-        <visual>
-            <origin rpy="0 0 0" xyz="0 0 0"/>
-            <geometry>
-                <box size="0.001 0.001 0.001"/>
-            </geometry>
-        </visual>
-    </link>
-    <joint name="floating_base_joint" type="fixed">
-        <origin rpy="0 0 0" xyz="0 0 0"/>
-        <parent link="world"/>
-        <child link="base"/>
-    </joint> -->
     <link name="base">
         <visual>
@@ -56,33 +43,8 @@
     </xacro:leg>
     <xacro:include filename="$(find realsense_ros_gazebo)/xacro/depthcam.xacro"/>
-    <!-- camera parameter for aliengo -->
-    <!-- <xacro:realsense_d435 sensor_name="d435_Forward" parent_link="base" rate="10">
-    <origin rpy="0 0 0 " xyz="0.31 0 0.03"/>
-    </xacro:realsense_d435>
-    <xacro:realsense_d435 sensor_name="d435_Back" parent_link="base" rate="10">
-    <origin rpy="0 0.9 3.14 " xyz="-0.34 0 0.05"/>
-    </xacro:realsense_d435> -->
-    <!-- 这个位置还可以 -->
-    <!-- <xacro:realsense_d435 sensor_name="d435_Down" parent_link="base" rate="10">
-    <origin rpy="0 0.85 0 " xyz="0.3 0 0.2"/>
-    </xacro:realsense_d435> -->
-    <!-- 试试把向下的摄像头位置加高看看效果 -->
-    <!-- <xacro:realsense_d435 sensor_name="d435_Down" parent_link="base" rate="10">
-    <origin rpy="0 1.0 0 " xyz="0.3 0 0.8"/>
-    </xacro:realsense_d435> -->
-    <!-- <xacro:realsense_d435 sensor_name="d435_Left" parent_link="base" rate="10">
-    <origin rpy="0 0.8 1.57 " xyz="0 0.08 0.06"/>
-    </xacro:realsense_d435>
-    <xacro:realsense_d435 sensor_name="d435_Right" parent_link="base" rate="10">
-    <origin rpy="0 0.8 -1.57 " xyz="0 -0.08 0.06"/>
-    </xacro:realsense_d435> -->
-    <!-- 好怪，有时候传感器加多了，地图反倒更加不稳定了 -->
     <!-- camera parameter for a1 -->
     <xacro:realsense_d435 sensor_name="camera" parent_link="base" rate="10">
     <origin rpy="0 0 0 " xyz="0.25 0 0.0"/>
     </xacro:realsense_d435>
-    <!-- <xacro:realsense_d435 sensor_name="d435_Back" parent_link="base" rate="10">
-    <origin rpy="0 0.9 3.14 " xyz="-0.25 0 0.05"/>
-    </xacro:realsense_d435> -->
     <xacro:realsense_d435 sensor_name="d435_Down" parent_link="base" rate="10">
     <origin rpy="0 0.7 0 " xyz="0.27 0 0.2"/>
@@ -97,10 +59,3 @@
   <xacro:include filename="$(find velodyne_description)/urdf/VLP-16.urdf.xacro" />   -->
     <!-- <xacro:arg name="simulation" default="false" /> -->
-    <!-- realsense和velodyne怎么不发布东西？ -->
-    <!-- <xacro:sensor_d435i parent="base" name="d435_Forward" use_nominal_extrinsics="$(arg simulation)">
-        <origin xyz="0.25 0.0 -0.009" rpy="0 0 0" />
-    </xacro:sensor_d435i>
-    <xacro:VLP-16 parent="base">
-        <origin xyz = "0.109 0.000 0.09" rpy="0 0 0" />
-    </xacro:VLP-16> -->
 </robot>
