Commit message: add reactive_gait

File: legged_examples/legged_unitree/legged_unitree_description/urdf/common/leg.xacro (robot description, xacro)
@@ -10,10 +10,8 @@
             <dynamics damping="${damping}" friction="${friction}"/>
             <xacro:if value="${(mirror_dae == True)}">
-                <limit effort="${hip_torque_max}" velocity="${hip_velocity_max}" lower="${hip_min}"
-                       upper="${hip_max}"/>
+                <limit effort="${hip_torque_max}" velocity="${hip_velocity_max}" lower="${hip_min}" upper="${hip_max}"/>
             </xacro:if>
             <xacro:if value="${(mirror_dae == False)}">
-                <limit effort="${hip_torque_max}" velocity="${hip_velocity_max}" lower="${-hip_max}"
-                       upper="${-hip_min}"/>
+                <limit effort="${hip_torque_max}" velocity="${hip_velocity_max}" lower="${-hip_max}" upper="${-hip_min}"/>
             </xacro:if>
         </joint>
@@ -59,6 +57,5 @@
             <axis xyz="0 1 0"/>
             <dynamics damping="${damping}" friction="${friction}"/>
-            <limit effort="${thigh_torque_max}" velocity="${thigh_velocity_max}" lower="${thigh_min}"
-                   upper="${thigh_max}"/>
+            <limit effort="${thigh_torque_max}" velocity="${thigh_velocity_max}" lower="${thigh_min}" upper="${thigh_max}"/>
         </joint>
         <link name="${prefix}_thigh">

File: legged_examples/legged_unitree/legged_unitree_description/urdf/robot.xacro (robot description, xacro)
@@ -17,4 +17,5 @@
             <origin rpy="0 0 0" xyz="0 0 0"/>
             <geometry>
+            <!--               0.267            0.194           0.114   -->
                 <box size="${trunk_length} ${trunk_width} ${trunk_height}"/>
             </geometry>
@@ -31,4 +32,5 @@
     <xacro:IMU connected_to="base" imu_name="unitree_imu" xyz="0. 0. 0." rpy="0. 0. 0."/>
     <xacro:leg prefix="RF" mirror="-1" mirror_dae="False" front_hind="1" front_hind_dae="True">
+    <!--                            0.1805              0.047   -->
         <origin rpy="0 0 0" xyz="${leg_offset_x} ${-leg_offset_y} 0"/>
     </xacro:leg>
@@ -44,12 +46,26 @@
     <xacro:include filename="$(find realsense_ros_gazebo)/xacro/depthcam.xacro"/>
     <!-- camera parameter for a1 -->
-    <xacro:realsense_d435 sensor_name="camera" parent_link="base" rate="10">
+    <xacro:realsense_d435 sensor_name="camera" parent_link="base" rate="50">
     <origin rpy="0 0 0 " xyz="0.25 0 0.0"/>
     </xacro:realsense_d435>
-    <xacro:realsense_d435 sensor_name="d435_Down" parent_link="base" rate="10">
+    <!-- <xacro:realsense_d435 sensor_name="d435_Down" parent_link="base" rate="10">
     <origin rpy="0 0.7 0 " xyz="0.27 0 0.2"/>
+    </xacro:realsense_d435> -->
+    <!-- <xacro:realsense_d435 sensor_name="d435_Down" parent_link="base" rate="50">
+    <origin rpy="0 0.6 0 " xyz="0.23 0 0.1"/>
+    </xacro:realsense_d435> -->
+    <!-- <xacro:realsense_d435 sensor_name="d435_Back" parent_link="base" rate="50">
+    <origin rpy="1.57 1.0 0 " xyz="-0.26 0 0.02"/>
+    </xacro:realsense_d435> -->
+    <!-- <xacro:realsense_d435 sensor_name="d435_Down" parent_link="base" rate="10">
+    <origin rpy="0 0.3 0 " xyz="0.108 0 0.137"/>
     </xacro:realsense_d435>
-    <!-- <xacro:include filename="$(find velodyne_description)/urdf/VLP-16.urdf.xacro"/> -->
-    <!-- <xacro:include filename="$(find velodyne_description)/urdf/HDL-32E.urdf.xacro"/> -->
+    <xacro:realsense_d435 sensor_name="d435_Left" parent_link="base" rate="10">
+    <origin rpy="0 0.3 1.0 " xyz="0.054 0.036 0.087"/>
+    </xacro:realsense_d435>
+    <xacro:realsense_d435 sensor_name="d435_Right" parent_link="base" rate="10">
+    <origin rpy="0 0.3 -1.0 " xyz="0.054 -0.036 0.087"/>
+    </xacro:realsense_d435> -->
+    <xacro:include filename="$(find lidar_description)/urdf/VLP-16.urdf.xacro"/>
     <!-- <xacro:VLP-16 name="VLP-16" parent="base">
     <origin rpy="0 0 0 " xyz="0.1 0 0.085 "/>
